Commit message: Update slam stuff

File: urdf/ld19.urdf (robot description, URDF)
Before this commit: robot ldlidar, 2 links, 1 joints
Links:
- removed link ldlidar_base
- removed link ldlidar_link
- added link laser; visual mesh filename=package://ld19_lidar/meshes/LD19.stl scale=0.001 0.001 0.001
- added link laser_link
Joints:
- removed joint ldlidar_link_joint
- added joint laser_link_joint: type fixed, parent laser, child laser_link, origin xyz=0 0 0.02745 rpy=0 0 0
